File: boards/03-usb-joystick/output/usb_joystick_routed.kicad_pcb (KiCad board)
At the start: 2 copper layers, 80 x 60 mm, 19 parts, among them J1 USB-C, J2 Joystick, SW1 Button, SW2 Button, SW3 Button, SW4 Button, U1 MCU, Y1 16MHz

Commit message: feat(optim): rotate edge-constrained connectors to face off-board (#4525)
* feat(optim): rotate edge-constrained connectors to face off-board

An `EdgeConstraint` could only translate a component toward its board
edge. A USB-C receptacle could therefore sit flush at the perimeter with
its plug opening aimed at the board interior -- placement the
EDGE_CONNECTOR_PLACEMENT check accepts but no cable can mate with. That
is exactly how board-03's J1 shipped: 7.6 mm inboard of the north edge,
mouth pointing at the buttons.

Library capability:

- `EdgeConstraint.mating_face_offset_deg` -- the off-board direction of a
  footprint's mating face in its own 0-degree frame (KiCad board frame,
  +Y = south). `None` keeps the pre-existing translation-only behavior.
- `compute_edge_orientation_torque()` -- torsion spring toward alignment
  with the assigned edge's outward `Edge.normal()`, summed into
  `PlacementOptimizer.compute_forces_and_torques()` alongside the
  existing 90-degree rotation-potential torque. Its magnitude saturates
  past 90 degrees of misalignment so the 180-degree (mouth-inward) case
  is not a zero-torque saddle.
- `edge_orientation_potential_energy()` -- added to `compute_energy()`,
  without which `run()` calls convergence (it samples linear velocity
  only) while a connector is still mid-flip.
- `snap_rotations()` resolves a hinted edge connector to the grid slot
  that faces off-board instead of the nearest one; the board boundary's
  own alignment torque has equal wells 180 degrees apart, so the discrete
  step is where the requirement has to be settled deterministically.
- `detect_edge_components(mating_faces=...)` / `from_pcb(mating_faces=...)`
  thread caller-supplied per-reference hints through.

board-03 consumes it:

- J1 rotated 180 degrees so the plug opening faces off the north edge,
  seated 0.5 mm inside Edge.Cuts, and given F.CrtYd artwork covering the
  real receptacle body -- without it the footprint claims to be only its
  pad field and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
Parts:
- moved J2 6.50 mm to (115.0, 92.5)
- moved J1 0.40 mm to (148.5, 65.9), turned to 180 degrees
Connections:
- U1 pad 27: USB_CC2 -> USB_CC1
- U1 pad 28: USB_D- -> USB_D+
- U1 pad 29: USB_D+ -> USB_D-
- U1 pad 30: USB_CC1 -> USB_CC2
Routing:
- net JOY_X: track 59.1 -> 78.5 mm
- net JOY_Y: track 54.1 -> 72.6 mm
- net JOY_BTN: track 26.2 -> 32.7 mm
- net USB_CC2: track 18.6 -> 21.5 mm, vias 0 -> 2
- net BTN3: track 19.7 -> 17.9 mm, vias 2 -> 0
- net USB_CC1: track 20.9 -> 19.2 mm, vias 2 -> 0
- net USB_D-: track 19.6 -> 20.2 mm
- net USB_D+: track 19.6 -> 20.2 mm
